Commit message: Ivanpauno/andino imu rebased (#265)
* Add Shell class

Signed-off-by: Javier Balloffet <javier.balloffet@gmail.com>

* Improve command prompt parsing

Signed-off-by: Javier Balloffet <javier.balloffet@gmail.com>

* Add dependencies for BNO055

Signed-off-by: Ivan Santiago Paunovic <ivanpauno@ekumenlabs.com>

* Added arduino code

Signed-off-by: Gonzalo de Pedro <gonzalo@depedro.com.ar>

Remove space

Signed-off-by: Gonzalo de Pedro <gonzalo@depedro.com.ar>

Added Imu to ros control

Signed-off-by: Gonzalo de Pedro <gonzalo@depedro.com.ar>

* Add ros2_control state interfaces for IMU

Signed-off-by: Ivan Santiago Paunovic <ivanpauno@ekumenlabs.com>

* fix random typo

Signed-off-by: Ivan Santiago Paunovic <ivanpauno@ekumenlabs.com>

* remove code not needed

Signed-off-by: Ivan Santiago Paunovic <ivanpauno@ekumenlabs.com>

* Fix sensor tag closure in xacro file.

* Add missing param

Signed-off-by: Ivan Santiago Paunovic <ivanpauno@ekumenlabs.com>

* Fix state interface imu data to read

Signed-off-by: Ivan Santiago Paunovic <ivanpauno@ekumenlabs.com>

* remove copied code

Signed-off-by: Ivan Santiago Paunovic <ivanpauno@ekumenlabs.com>

* Spawn imu controller

Signed-off-by: Ivan Santiago Paunovic <ivanpauno@ekumenlabs.com>

* fix

Signed-off-by: Ivan Santiago Paunovic <ivanpauno@ekumenlabs.com>

* Fix state interface names (maybe)

Signed-off-by: Ivan Santiago Paunovic <ivanpauno@ekumenlabs.com>

* Same for ros control urdf

Signed-off-by: Ivan Santiago Paunovic <ivanpauno@ekumenlabs.com>

* Fix post rebasing errors

Signed-off-by: Ivan Santiago Paunovic <ivanpauno@ekumenlabs.com>

* Add Arduino IDE dependencies in README

Signed-off-by: Ivan Santiago Paunovic <ivanpauno@ekumenlabs.com>

* Gazebo changes

Signed-off-by: Gonzalo de Pedro <gonzalo@depedro.com.ar>

* andino urdf

Signed-off-by: Gonzalo de Pedro <gonzalo@depedro.com.ar>

* Fixed dangling conflicts

Signed-off-by: Gonzalo de Pedro <gonzalo@depedro.com.ar>

* Added commands for imu

Signed-off-by: Gonzalo de Pedro <gonzalo@depedro.com.ar>

* Fixed has imu command variable name

Signed-off-by: Gonzalo de Pedro <gonzalo@depedro.com.ar>

* Remove andino firmware changes

Signed-off-by: Gonzalo de Pedro <gonzalo@depedro.com.ar>

---------

Signed-off-by: Javier Balloffet <javier.balloffet@gmail.com>
Signed-off-by: Ivan Santiago Paunovic <ivanpauno@ekumenlabs.com>
Signed-off-by: Gonzalo de Pedro <gonzalo@depedro.com.ar>
Co-authored-by: Ivan Santiago Paunovic <ivanpauno@ekumenlabs.com>
Co-authored-by: Gonzalo de Pedro <gonzalo@depedro.com.ar>
Co-authored-by: fbaglivo <fbaglivo@ekumenlabs.com>

File: andino_description/urdf/andino.urdf.xacro (robot description, xacro)
@@ -63,9 +63,11 @@
   </xacro:motor>
   <!-- Sensors -->
-  <xacro:laser prefix="rplidar" parent_link="second_base_link"
+  <xacro:laser prefix="rplidar" parent_link="base_link"
                    sensor_prop="${sensor_prop}">
   </xacro:laser>
   <xacro:camera_sensor parent_link="base_link" sensor_prop="${sensor_prop}">
   </xacro:camera_sensor>
+  <xacro:imu_sensor parent_link="base_link" sensor_prop="${sensor_prop}">
+  </xacro:imu_sensor>
   <!-- ros2_control -->
   <xacro:if value="$(arg use_real_ros_control)">

File: andino_description/urdf/include/andino_control.urdf.xacro (robot description, xacro)
@@ -1,37 +1,45 @@
 <?xml version="1.0"?>
 <robot xmlns:xacro="http://www.ros.org/wiki/xacro">
-<!-- ===================== Control xacro =========================================
-  params:
-  - hardware_props [dictionary]: hardware properties loaded from the YAML file.
--->
-  <xacro:macro name="control" params="hardware_props" >
-    <!-- TODO(francocipollone): This xacro should be part of andino_control package instead.-->
-    <ros2_control name="RealRobot" type="system">
-      <hardware>
-        <plugin>andino_base/DiffDriveAndino</plugin>
-        <param name="left_wheel_name">${hardware_props['left_wheel_name']}</param>
-        <param name="right_wheel_name">${hardware_props['right_wheel_name']}</param>
-        <param name="serial_device">${hardware_props['serial_device']}</param>
-        <param name="baud_rate">${hardware_props['baud_rate']}</param>
-        <param name="timeout">${hardware_props['timeout']}</param>
-        <param name="enc_ticks_per_rev">${hardware_props['enc_ticks_per_rev']}</param>
-      </hardware>
-      <joint name="left_wheel_joint">
-        <command_interface name="velocity">
-          <param name="min">-5</param>
-          <param name="max">5</param>
-        </command_interface>
-        <state_interface name="velocity"/>
-        <state_interface name="position"/>
-      </joint>
-      <joint name="right_wheel_joint">
-        <command_interface name="velocity">
-          <param name="min">-5</param>
-          <param name="max">5</param>
-        </command_interface>
-        <state_interface name="velocity"/>
-        <state_interface name="position"/>
-      </joint>
-    </ros2_control>
-  </xacro:macro>
+  <!-- TODO(francocipollone): This xacro should be part of andino_control package instead.-->
+  <ros2_control name="RealRobot" type="system">
+    <hardware>
+      <plugin>andino_base/DiffDriveAndino</plugin>
+      <!-- TODO(francocipollone): Parameters like loop_rate, device, baud_rate, etc should be loaded from a file or passed via the launch file as xacro args -->
+      <param name="left_wheel_name">left_wheel_joint</param>
+      <param name="right_wheel_name">right_wheel_joint</param>
+      <param name="serial_device">/dev/ttyUSB_ARDUINO</param>
+      <param name="baud_rate">57600</param>
+      <param name="timeout">1000</param>
+      <param name="enc_ticks_per_rev">585</param>
+      <param name="imu_sensor_name">imu_sensor</param>
+    </hardware>
+    <joint name="left_wheel_joint">
+      <command_interface name="velocity">
+        <param name="min">-5</param>
+        <param name="max">5</param>
+      </command_interface>
+      <state_interface name="velocity"/>
+      <state_interface name="position"/>
+    </joint>
+    <joint name="right_wheel_joint">
+      <command_interface name="velocity">
+        <param name="min">-5</param>
+        <param name="max">5</param>
+      </command_interface>
+      <state_interface name="velocity"/>
+      <state_interface name="position"/>
+    </joint>
+    <sensor name="imu_sensor">
+      <state_interface name="orientation.x"/>
+      <state_interface name="orientation.y"/>
+      <state_interface name="orientation.z"/>
+      <state_interface name="orientation.w"/>
+      <state_interface name="angular_velocity.x"/>
+      <state_interface name="angular_velocity.y"/>
+      <state_interface name="angular_velocity.z"/>
+      <state_interface name="linear_acceleration.x"/>
+      <state_interface name="linear_acceleration.y"/>
+      <state_interface name="linear_acceleration.z"/>
+    </sensor>
+  </ros2_control>
 </robot>

File: andino_description/urdf/include/common_sensors.urdf.xacro (robot description, xacro)
@@ -84,3 +84,32 @@
   </joint>
 </xacro:macro>
+<xacro:macro name="imu_sensor" params="parent_link sensor_prop">
+  <link name="imu_link">
+    <visual>
+      <origin xyz="0 0 0" rpy="0 0 0"/>
+      <geometry>
+        <box size="${sensor_prop['imu']['box_size']} ${sensor_prop['imu']['box_size']} ${sensor_prop['imu']['box_size_height']}"/>
+      </geometry>
+      <material name="black"/>
+    </visual>
+    <collision>
+      <origin xyz="0 0 0" rpy="0 0 0"/>
+      <geometry>
+        <box size="${sensor_prop['imu']['box_size']} ${sensor_prop['imu']['box_size']} ${sensor_prop['imu']['box_size_height']}"/>
+      </geometry>
+    </collision>
+    <xacro:box_inertia m="${sensor_prop['imu']['mass']}"
+                            x="${sensor_prop['imu']['box_size']}"
+                            y="${sensor_prop['imu']['box_size']}"
+                            z="${sensor_prop['imu']['box_size_height']}"
+                            o_xyz="0 0 0"
+                            o_rpy="0 0 0" />
+  </link>
+  <joint name="imu_joint" type="fixed">
+    <parent link="${parent_link}"/>
+    <child link="imu_link"/>
+    <origin xyz="${sensor_prop['imu']['dx']} ${sensor_prop['imu']['dy']} ${sensor_prop['imu']['dz']}" rpy="0 0 0"/>
+    <axis xyz="0 1 0" />
+  </joint>
+</xacro:macro>
 </robot>

File: andino_gz_classic/urdf/andino_gz_classic.xacro (robot description, xacro)
@@ -138,4 +138,59 @@
         </sensor>
   </gazebo>
+  <gazebo reference="imu_link">
+      <sensor name="imu" type="imu">
+          <always_on>true</always_on>
+          <update_rate>100</update_rate>
+          <imu>
+            <angular_velocity>
+              <x>
+                <noise type="gaussian">
+                  <mean>0.0</mean>
+                  <stddev>2e-4</stddev>
+                </noise>
+              </x>
+              <y>
+                <noise type="gaussian">
+                  <mean>0.0</mean>
+                  <stddev>2e-4</stddev>
+                </noise>
+              </y>
+              <z>
+                <noise type="gaussian">
+                  <mean>0.0</mean>
+                  <stddev>2e-4</stddev>
+                </noise>
+              </z>
+            </angular_velocity>
+            <linear_acceleration>
+              <x>
+                <noise type="gaussian">
+                  <mean>0.0</mean>
+                  <stddev>1.7e-2</stddev>
+                </noise>
+              </x>
+              <y>
+                <noise type="gaussian">
+                  <mean>0.0</mean>
+                  <stddev>1.7e-2</stddev>
+                </noise>
+              </y>
+              <z>
+                <noise type="gaussian">
+                  <mean>0.0</mean>
+                  <stddev>1.7e-2</stddev>
+                </noise>
+              </z>
+            </linear_acceleration>
+          </imu>
+          <plugin name="imu_plugin" filename="libgazebo_ros_imu_sensor.so">
+              <ros>
+                  <namespace>imu</namespace>
+                  <remapping>~/out:=data</remapping>
+              </ros>
+              <initial_orientation_as_reference>false</initial_orientation_as_reference>
+          </plugin>
+      </sensor>
+  </gazebo>
   <xacro:include filename="$(find andino_gz_classic)/urdf/include/andino_materials.xacro"/>
 </robot>
